Commit message: Capture Go2 baseline progress for desktop testing
Preserve Jazzy CHAMP sources, walking evidence, migration instructions and legacy runtime scripts. Keep ongoing performance work explicitly unverified. VM disks and runtime credentials remain external.

File: unitree_ros-master/robots/go2_description/xacro/robot.xacro (robot description, xacro)
@@ -37,5 +37,5 @@
             <origin rpy="0 0 0" xyz="0 0 0"/>
             <geometry>
-                <mesh filename="package://go2_description/meshes/trunk.dae" scale="1 1 1"/>
+                <mesh filename="package://go2_description/meshes/base.dae" scale="1 1 1"/>
             </geometry>
             <!-- <material name="orange"/> -->
