Commit message: Preserve in-progress Go2 RGB-D, lidar and feedback odometry work
User requested stopping laptop development and handing current code to desktop.
Sensor integration is incomplete; retain failed trials and do not mark accepted.

File: baseline/go2_jazzy/vendor/unitree_go2_description/urdf/lidar_4D_lidar.xacro (robot description, xacro)
@@ -4,9 +4,5 @@
         <!-- Lidar L1-->
         <link name="lidar_l1_link">
-            <inertial>
-                <mass value="0.5"/>
-                <origin rpy="0 0 0" xyz="0 0 0"/>
-                <inertia ixx="0.01" ixy="0" ixz="0" iyy="0.01" iyz="0" izz="0.01"/>
-            </inertial>
+            <!-- Onboard measurement frame; no additional payload mass or collision. -->
             <visual>
                 <origin rpy="0 0 0" xyz="0 0 0"/>
@@ -18,13 +14,4 @@
                 </material>
             </visual>
-            <collision>
-                <origin rpy="0 0 0" xyz="0 0 0"/>
-                <geometry>
-                    <mesh filename="file://$(find unitree_go2_description)/meshes/L1_4D_Lidar.dae" scale="1 1 1"/>
-                </geometry>
-                <material name="black">
-                    <color rgba="0.0 0.0 0.0 1.0"/>
-                </material>
-            </collision>
         </link>
         <joint name="lidar_l1_joint" type="fixed">
@@ -37,9 +24,9 @@
             <sensor name="lidar_l1" type="gpu_lidar">
                 <topic>unitree_lidar</topic>
-                <update_rate>10</update_rate>
+                <update_rate>$(arg lidar_rate)</update_rate>
                 <lidar>
                     <scan>
                         <horizontal>
-                            <samples>600</samples>
+                            <samples>$(arg lidar_samples)</samples>
                             <resolution>1</resolution>
                             <min_angle>-3.14159</min_angle>
@@ -47,5 +34,5 @@
                         </horizontal>
                         <vertical>
-                            <samples>30</samples>
+                            <samples>$(arg lidar_channels)</samples>
                             <resolution>1</resolution>
                             <min_angle>-0.785398</min_angle>

File: baseline/go2_jazzy/vendor/unitree_go2_description/urdf/realsense_d455.xacro (robot description, xacro)
@@ -1,33 +1,31 @@
 <?xml version="1.0"?>
 <robot xmlns:xacro="http://www.ros.org/wiki/xacro">
-    <!-- Include the RealSense D455 URDF macro from realsense2_description -->
-    <xacro:include filename="$(find realsense2_description)/urdf/_d455.urdf.xacro"/>
-    <xacro:macro name="d455_camera">
-        <!-- Mount the D455 on top of the trunk, in front of the velodyne lidar -->
-        <xacro:sensor_d455 parent="trunk" name="d455_camera" use_nominal_extrinsics="true">
-            <origin xyz="0.28 0 0.062" rpy="0 0 0"/>
-        </xacro:sensor_d455>
-        <!-- Gazebo Sim RGBD Camera sensor plugin -->
-        <gazebo reference="d455_camera_link">
-            <sensor name="d455_rgbd_camera" type="rgbd_camera">
-                <pose>0 0 0 0 0 0</pose>
-                <camera>
-                    <horizontal_fov>1.489</horizontal_fov>
-                    <image>
-                        <width>640</width>
-                        <height>480</height>
-                    </image>
-                    <clip>
-                        <near>0.1</near>
-                        <far>10.0</far>
-                    </clip>
-                </camera>
-                <always_on>1</always_on>
-                <update_rate>15</update_rate>
-                <visualize>true</visualize>
-                <topic>d455</topic>
-                <gz_frame_id>d455_camera_link</gz_frame_id>
-            </sensor>
-        </gazebo>
-    </xacro:macro>
+  <!-- Idealized RGB-D simulation; not a calibrated RealSense hardware emulator. -->
+  <xacro:macro name="d455_camera">
+    <link name="d455_camera_link">
+            <!-- Onboard measurement frame; no additional payload mass or collision. -->
+      <visual><geometry><box size="0.025 0.124 0.029"/></geometry><material name="black"/></visual>
+    </link>
+    <joint name="d455_camera_joint" type="fixed">
+      <parent link="trunk"/><child link="d455_camera_link"/>
+      <origin xyz="0.28 0 0.062" rpy="0 0 0"/>
+    </joint>
+    <link name="d455_camera_optical_frame"/>
+    <joint name="d455_camera_optical_joint" type="fixed">
+      <parent link="d455_camera_link"/><child link="d455_camera_optical_frame"/>
+      <origin xyz="0 0 0" rpy="-1.57079632679 0 -1.57079632679"/>
+    </joint>
+    <gazebo reference="d455_camera_link">
+      <sensor name="d455_rgbd_camera" type="rgbd_camera">
+        <camera>
+          <horizontal_fov>1.489</horizontal_fov>
+          <image><width>$(arg camera_width)</width><height>$(arg camera_height)</height><format>R8G8B8</format></image>
+          <clip><near>0.1</near><far>10.0</far></clip>
+        </camera>
+        <always_on>true</always_on><update_rate>$(arg camera_rate)</update_rate>
+        <visualize>false</visualize><topic>d455</topic>
+        <gz_frame_id>d455_camera_optical_frame</gz_frame_id>
+      </sensor>
+    </gazebo>
+  </xacro:macro>
 </robot>

File: baseline/go2_jazzy/vendor/unitree_go2_description/urdf/unitree_go2_robot.xacro (robot description, xacro)
@@ -11,4 +11,10 @@
     <xacro:arg name="disable_lidar_l1" default="false"/>
     <xacro:arg name="disable_velodyne_lidar" default="false"/>
+    <xacro:arg name="camera_width" default="640"/>
+    <xacro:arg name="camera_height" default="480"/>
+    <xacro:arg name="camera_rate" default="15"/>
+    <xacro:arg name="lidar_samples" default="600"/>
+    <xacro:arg name="lidar_channels" default="30"/>
+    <xacro:arg name="lidar_rate" default="10"/>
     <xacro:include filename="$(find unitree_go2_description)/urdf/const.xacro" />
     <xacro:include filename="$(find unitree_go2_description)/urdf/materials.xacro" />
